File: MaD_Edge_Sheet3.kicad_sch (KiCad schematic)
At the start: 46 parts, among them IC14 ISO6741DWR, IC15 ISO6721BDR, IC16 ISO6740FDWR, J20 Encoder, J21 ServoCtrl, J23 ServoSerial, Q1 NPN, U24 AM26LS31CD, U25 AM26LV32xD, U27 SN74LVC1G14DBV, U28 SN74LVC1G14DBV, U29 SN74LVC1G14DBV, U30 SN74LVC1G14DBV, U31 SN74LVC1G14DBV, U32 SN74LVC1G14DBV, U33 SN74LVC1G14DBV, U34 SN74LVC1G14DBV

Commit message: working version for getting basic data for the thesis
Parts:
- C24, C25, C26, C27, C28, C29, R24, R25: Qty Bought (none) -> 100 - lcsc
- D18, D19, D20, D21, D22, D23, D24, D25: Qty Bought (none) -> 80 - lcsc
- IC14, IC16: Qty Bought (none) -> 3 - lcsc
- IC15: Qty Bought (none) -> 4 - lscs
- J20: Qty Bought (none) -> 6 digikey; Receptical (none) -> 0430251000
- J21: Receptical (none) -> 0430251000
- JP1, JP2, JP3, JP4, JP5: Qty Bought (none) -> header
- Q1: Qty Bought (none) -> 50 - lcsc
- R30, R31, R32, R33, R34, R35, R36, R37: Qty Bought (none) -> 200 - lcsc
- U24: Qty Bought (none) -> 4 lcsc
- U25: Qty Bought (none) -> 3 lcsc
- U27, U28, U29, U30, U31, U32, U33, U34: Qty Bought (none) -> 100 lcsc
